File: Eco-PCB-2/Eco-PCB-2.kicad_pcb (KiCad board)
At the start: 2 copper layers, 15 parts, among them J1 DB25_Female, J2 Switch, P1 Push Button, P2 Push Button

Commit message: updated pin sizes issue and spacing on PCB2
Parts:
- moved D4 15.2 mm to (95.2, 119.6)
- moved D3 11.8 mm to (95.2, 112.6)
- moved D2 7.49 mm to (95.2, 104.4)
- moved D1 3.42 mm to (95.2, 96.7)
- moved P1 2.74 mm to (93.4, 97.6)
Routing:
- net VCC: track 139.6 -> 197.0 mm
- net CLK: track 30.6 -> 42.5 mm
- net GND: track 131.6 -> 141.7 mm
- net D4: track 23.1 -> 29.5 mm
- net D3: track 22.7 -> 27.7 mm
- net D2: track 23.0 -> 25.5 mm
- net D1: track 22.9 -> 24.4 mm
- net Net-(P1-Pad1): track 5.36 -> 6.51 mm
Other:
- board text added: "SEM"
